File: A-ESTF_V2_EP4CE22Board/Hardware/IOConns/IOConns/IOConns.sch (KiCad schematic (older format))
At the start: 5 parts, among them J10 Conn_02x20_Odd_Even, J3 Conn_01x03, J4 Conn_01x03, J5 Conn_01x20

Commit message: io conns
Other:
- note added: "Pin 2 next to\nJ10 silkscreen"
- note removed: "Pin 1 next to\nJ10 silkscreen"
Changed lines of the file:
@@
 Text Notes 7100 4500 0    50   ~ 0
 Pin 1 next to\nJ5 silkscreen
-Text Notes 4950 4500 0    50   ~ 0
-Pin 1 next to\nJ10 silkscreen
+Text Notes 6000 4500 0    50   ~ 0
+Pin 2 next to\nJ10 silkscreen
 Text Notes 8800 4300 0    50   ~ 0
 LCD (ref)

Commit message: Shuffle files
Connections:
- net labels added: LCD_VCC
Changed lines of the file:
@@
 Text Notes 8800 4300 0    50   ~ 0
 LCD (ref)
+Text Label 6150 4300 0    50   ~ 0
+LCD_VCC
+Text Label 5000 4300 0    50   ~ 0
+LCD_VCC
 $EndSCHEMATC

Commit message: FPGA Card docs
Connections:
- net labels added: PIN_E10, PIN_F14, PIN_K16, PIN_L14, PIN_L16, PIN_R11, PIN_T11
- wire segments 63 -> 57
- no-connect marks 0 -> 8
Other:
- note added: "IO_0"
- note added: "IO_1"
- note added: "IO_10"
- note added: "IO_11"
- note added: "IO_12"
- note added: "IO_13"
- note added: "IO_14"
- note added: "IO_15"
- note added: "IO_16"
- note added: "IO_17"
- note added: "IO_18"
- note added: "IO_19"
- note added: "IO_2"
- note added: "IO_20"
- note added: "IO_21"
- note added: "IO_22"
- note added: "IO_23"
- note added: "IO_3"
- note added: "IO_4"
- note added: "IO_5"
- note added: "IO_6"
- note added: "IO_7"
- note added: "IO_8"
- note added: "IO_9"
- moved on the sheet: J10, J3, J4, U?
